Commit message: nav2 params

File: urdf/ackermann_robot.xacro (robot description, xacro)
@@ -1,22 +1,24 @@
 <?xml version="1.0"?>
 <robot name="ackermann_bot" xmlns:xacro="http://www.ros.org/wiki/xacro">
-  <xacro:property name="wheelbase" value="0.5"/>
-  <xacro:property name="track_width" value="0.4"/>
+  <xacro:property name="wheelbase" value="0.5"/>   <!-- Distance between front and rear axle -->
+  <xacro:property name="track_width" value="0.4"/> <!-- Distance between left and right wheels -->
   <xacro:property name="wheel_radius" value="0.1"/>
+  <!-- Base Link -->
   <link name="base_link">
     <visual>
       <geometry>
-        <box size="0.5 0.3 0.2"/>
+        <box size="0.5 0.3 0.2"/> <!-- Body of the robot -->
       </geometry>
       <material name="blue"/>
     </visual>
   </link>
-  <joint name="base_to_front_wheel" type="continuous">
+  <!-- Front Left Wheel -->
+  <joint name="front_left_steering_joint" type="continuous">
     <parent link="base_link"/>
-    <child link="front_wheel"/>
-    <origin xyz="0.25 0 0"/>
-    <axis xyz="0 0 1"/>
+    <child link="front_left_wheel"/>
+    <origin xyz="${wheelbase/2} ${track_width/2} 0"/>
+    <axis xyz="0 0 1"/>  <!-- Steering rotation along Z-axis -->
   </joint>
-  <link name="front_wheel">
+  <link name="front_left_wheel">
     <visual>
       <geometry>
@@ -25,10 +27,66 @@
     </visual>
   </link>
-  <joint name="base_to_rear_wheel" type="fixed">
+  <joint name="front_left_wheel_joint" type="continuous">
+    <parent link="front_left_wheel"/>
+    <child link="front_left_tire"/>
+    <origin xyz="0 0 0"/>
+    <axis xyz="0 1 0"/>  <!-- Rolling motion along Y-axis -->
+  </joint>
+  <link name="front_left_tire">
+    <visual>
+      <geometry>
+        <cylinder length="0.02" radius="${wheel_radius}"/>
+      </geometry>
+    </visual>
+  </link>
+  <!-- Front Right Wheel -->
+  <joint name="front_right_steering_joint" type="continuous">
     <parent link="base_link"/>
-    <child link="rear_wheel"/>
-    <origin xyz="-0.25 0 0"/>
+    <child link="front_right_wheel"/>
+    <origin xyz="${wheelbase/2} -${track_width/2} 0"/>
+    <axis xyz="0 0 1"/>  <!-- Steering rotation along Z-axis -->
   </joint>
-  <link name="rear_wheel">
+  <link name="front_right_wheel">
+    <visual>
+      <geometry>
+        <cylinder length="0.02" radius="${wheel_radius}"/>
+      </geometry>
+    </visual>
+  </link>
+  <joint name="front_right_wheel_joint" type="continuous">
+    <parent link="front_right_wheel"/>
+    <child link="front_right_tire"/>
+    <origin xyz="0 0 0"/>
+    <axis xyz="0 1 0"/>  <!-- Rolling motion along Y-axis -->
+  </joint>
+  <link name="front_right_tire">
+    <visual>
+      <geometry>
+        <cylinder length="0.02" radius="${wheel_radius}"/>
+      </geometry>
+    </visual>
+  </link>
+  <!-- Rear Left Wheel -->
+  <joint name="rear_left_wheel_joint" type="continuous">
+    <parent link="base_link"/>
+    <child link="rear_left_wheel"/>
+    <origin xyz="-${wheelbase/2} ${track_width/2} 0"/>
+    <axis xyz="0 1 0"/>  <!-- Rolling motion along Y-axis -->
+  </joint>
+  <link name="rear_left_wheel">
+    <visual>
+      <geometry>
+        <cylinder length="0.02" radius="${wheel_radius}"/>
+      </geometry>
+    </visual>
+  </link>
+  <!-- Rear Right Wheel -->
+  <joint name="rear_right_wheel_joint" type="continuous">
+    <parent link="base_link"/>
+    <child link="rear_right_wheel"/>
+    <origin xyz="-${wheelbase/2} -${track_width/2} 0"/>
+    <axis xyz="0 1 0"/>  <!-- Rolling motion along Y-axis -->
+  </joint>
+  <link name="rear_right_wheel">
     <visual>
       <geometry>
